File: Tympan nRF52 Programmer/Tympan nRF52 Programmer.kicad_pcb (KiCad board)
At the start: 2 copper layers, 38 x 74 mm, 5 parts, among them J2 FTSH-105-01-L-DV-K, J7 J-Link, P6 CONN_01X01, P7 CONN_01X01, P8 CONN_01X01

Commit message: Production Files Approved
Parts:
- added G***: LOGO, Solutions:Tympan_LOGO, F.Cu at (152.9, 97.2)
- added G***: LOGO, Solutions:Flywheel, F.Cu at (152.4, 80.7)
- added P1: CONN_01X01, MountingHole:MountingHole_3mm, F.Cu at (126.9, 130.7)
- J2: footprint Tympan:SAMTEC_FTSH-105-01-L-DV-K -> Tympan:SAMTEC_SHF-105-01-X-D-TH
- J7: footprint Solutions:J-Link_SMT_SIP_0.1inP -> Tympan:J-Link_POGO_SIP_0.1inP
- moved J2 28.3 mm to (126.3, 116.2), turned to -90 degrees
Routing:
- net /BT_nRESET: track 0.20 -> 36.6 mm
- net /SWO: track 0.00 -> 26.9 mm
- net /SWCLK: track 0.00 -> 19.9 mm
- net +3.3V: track 0.00 -> 17.3 mm
- net /SWDIO: track 0.00 -> 9.84 mm
- removed copper zone on B.Cu, net +3.3V
Other:
- board size 38 x 74 mm -> 55 x 79 mm
- board text added: "Tympan Rev F nRF52 Boot Loader Fixture"
- board text removed: "Designed by Flywheel Lab Brooklyn, NY"
- board text removed: "GND +BATT SW_BAT 34 35"
- board text removed: "INPUT"
- board text removed: "LEFT"
- board text removed: "OUTPUT"
- board text removed: "PROGRAM"
- board text removed: "RIGHT"
- board text removed: "Tympan Rev F"
- board text removed: "tympan.org"
